File: arduino_brainmachine.kicad_sch (KiCad schematic)
At the start: 38 parts, among them Q1 2N5551, Q2 2N5551

Commit message: Upgrade
Parts:
- added R21: 220 Om, symbol PCM_Elektuur:R
- added SW1: SW_Push, symbol Switch:SW_Push
Connections:
- net GND: now also A1.GND6 (GND), SW1.2
- net at A1.D0 (D0/RX0): now also R21.2 (-)
- net at A1.D2 (D2_INT0): now also R21.1 (+), SW1.1

Commit message: Upgrade
Connections:
- net at D1.2 (A): now also A1.5V4 (5V), D2.2 (A); no longer R1.1 (+)
- net at R2.1 (+): now also D2.1 (K); no longer D2.2 (A)
- new net: D1.1 (K), R1.1 (+)
Other:
- moved on the sheet: D1, D2

Commit message: Upgrade
Parts:
- removed C6, C8: 1 mkF, symbol PCM_Elektuur:C
- added D3: 12 v, symbol Device:D_Zener
- added R22, R23: 47 Om, symbol PCM_Elektuur:R
- C1, C3, C5, C7: value 1 mkF -> 10 mkF
- R10, R12: value 47 Om -> 1 kOm
- R5, R6: value 4.7 Om -> 1 kOm
Connections:
- net +12V: now also D3.1 (K)
- net GND: now also R10.1 (+), R12.1 (+), R5.1 (+), R6.1 (+); no longer C1.2 (-), C3.2 (-)
- net JLH Class-A L or R Channel: now also C2.1 (+), C4.1 (+), R3.2 (-), R4.2 (-); no longer Q1.3 (C), Q2.3 (C), R16.2 (-), R17.2 (-)
- net PC/Other: now also C1.1 (+), C3.1 (+); no longer R5.2 (-), R6.2 (-)
- net at C7.2 (-), R11.1 (+): now also R6.2 (-)
- net at Q2.2 (B), R11.2 (-), R18.1 (+)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: now also R4.1 (+), R23.2 (-); no longer R12.2 (-)
- net at Q1.2 (B), R13.1 (+), R15.2 (-)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: now also R22.2 (-); no longer R10.2 (-)
- net at RV5.1: now also C5.1 (+); no longer R4.1 (+)
- net at RV5.4: now also C7.1 (+); no longer R3.1 (+)
- net at C5.2 (-), R9.1 (+): now also R5.2 (-)
- new net: C1.2 (-), R12.2 (-), R23.1 (+)
- new net: Q2.3 (C), R16.2 (-)
- new net: C3.2 (-), R10.2 (-), R22.1 (+)
- new net: Q1.3 (C), R17.2 (-), R3.1 (+)
- new net Earth: D3.2 (A)

Commit message: Upgrade
Parts:
- added C6, C8: 1 mkF, symbol PCM_Elektuur:C
- added MK1: Microphone_Condenser, symbol Device:Microphone_Condenser
- added Q3: 2N5551, Package_TO_SOT_THT:TO-39-3, symbol Transistor_BJT:2N2219
- added R24: 330 Om, symbol PCM_Elektuur:R
- added R25: 200 Om, symbol PCM_Elektuur:R
- added R26, R28: 2 KOm, symbol PCM_Elektuur:R
- added R27: 1.2 KOm, symbol PCM_Elektuur:R
- added R29: 4.7 Om, symbol PCM_Elektuur:R
Connections:
- net +12V: now also R26.2 (-), R27.1 (+), R28.2 (-)
- net GND: now also C8.2 (-), MK1.1 (-), R24.1 (+), R25.1 (+)
- net at A1.A0: now also RV1.2
- net at A1.A1: now also RV2.2; no longer RV1.2
- net at A1.A2: now also RV3.2; no longer RV2.2
- net at A1.A3: now also RV4.2; no longer RV3.2
- net at A1.A4: now also C8.1 (+), R29.2 (-); no longer RV4.2
- net OCR0A = ((-t & 4095) * (255 & t * (t & t >> 13)) >> 12) + (127 & t * (234 & t >> 8 & t >> 3) >> (3 & t >> 14)); WIP: no longer names the net of A1.D13
- new net: C6.1 (+), MK1.2 (+), R28.1 (+)
- new net: C6.2 (-), Q3.2 (B), R24.2 (-), R26.1 (+)
- new net: Q3.3 (C), R27.2 (-), R29.1 (+)
- new net: Q3.1 (E), R25.2 (-)
Other:
- note added: "https://github.com/asciiscry3r/brainmachine/tree/main/sketch_dec12a"

Commit message: Upgrade
Parts:
- R28: value 2 KOm -> 33-56 KOm
Changed lines of the file:
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@@
 			)
 		)
-		(property "Value" "2 KOm"
+		(property "Value" "33-56 KOm"
 			(at 49.53 127 90)
 			(effects

Commit message: Upgrade
Parts:
- R28: value 33-56 KOm -> 30-56 KOm
Connections:
- net +5V: no longer RV2.1, RV4.1
- net GND: no longer RV1.3, RV3.3
- net at A1.A0, RV1.2: now also RV1.3, RV2.1, RV2.2
- net at A1.A1: now also RV3.2, RV3.3, RV4.1, RV4.2; no longer RV2.2
- net at A1.A2: now also C8.1 (+), R29.2 (-); no longer RV3.2
- net at A1.A3: no longer RV4.2
- now unconnected: A1.A4

Commit message: update
Parts:
- added C10: 10-100mkF, symbol PCM_Elektuur:C-polar
- added C9: 1000mkF, symbol PCM_Elektuur:C-polar
- added D4: LED, symbol Device:LED
- added Q4: 2N5551, Package_TO_SOT_THT:TO-39-3, symbol Transistor_BJT:2N2219
- added R30: 1 kOm, symbol PCM_Elektuur:R
- added R31, R33: 1-10 KOm, symbol PCM_Elektuur:R
- added R32: 91 KOm, symbol PCM_Elektuur:R
- added R34: 1 KOm, symbol Device:R_Small
Connections:
- net +5V: now also C10.1 (+), Q4.3 (C), R32.2 (-)
- net GND: now also C9.2 (-), D4.1 (K), R31.1 (+), R33.1 (+)
- net at A1.D4: now also R30.1 (+)
- new net: Q4.2 (B), R30.2 (-), R32.1 (+)
- new net: C9.1 (+), Q4.1 (E), R33.2 (-), R34.1
- new net: D4.2 (A), R34.2
- new net: C10.2 (-), R31.2 (-)

Commit message: Upgrade
Parts:
- added Q5, Q6: PNP, symbol Simulation_SPICE:PNP
- added R35, R36: 900 Om, symbol PCM_Elektuur:R
- added U1, U2: VOS618A, Package_SO:SSOP-4_4.4x2.6mm_P1.27mm, symbol Isolator:VOS618A
Connections:
- net at A1.5V4 (5V), D1.2 (A), D2.2 (A): now also Q5.3 (E), Q6.3 (E), U1.1, U2.1
- net at A1.D12: now also R35.1 (+)
- net at A1.D13: now also R36.1 (+)
- net at A1.D4, R30.1 (+): now also A1.D5, A1.D6, R1.2 (-), R2.2 (-)
- new net: Q6.2 (B), R36.2 (-), U1.2
- new net: Q5.2 (B), R35.2 (-), U2.2
Other:
- moved on the sheet: D1, D2, R1, R2
