File: arduino_brainmachine.kicad_sch (KiCad schematic)
At the start: 66 parts, among them Q1 2N5551, Q2 2N5551, Q3 2N5551, Q4 2N5551, Q5 PNP, Q6 PNP, SW1 SW_Push, U1 VOS618A, U2 VOS618A

Commit message: Upgrade
Other:
- added sheet Untitled Sheet (untitled.kicad_sch)
Changed lines of the file:
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@@
 	(generator_version "8.0")
 	(paper "A4")
+	(title_block
+		(date "2025-02-18")
+	)
 	(junction
 		(at 40.64 96.52)
@@
 		)
 	)
+	(sheet
+		(at 306.07 2.54)
+		(size 280.67 203.2)
+		(fields_autoplaced yes)
+		(stroke
+			(width 0.1524)
+			(type solid)
+		)
+		(fill
+			(color 0 0 0 0.0000)
+		)
+		(property "Sheetname" "Untitled Sheet"
+			(at 306.07 1.8284 0)
+			(effects
+				(font
+					(size 1.27 1.27)
+				)
+				(justify left bottom)
+			)
+		)
+		(property "Sheetfile" "untitled.kicad_sch"
+			(at 306.07 206.3246 0)
+			(effects
+				(font
+					(size 1.27 1.27)
+				)
+				(justify left top)
+			)
+		)
+		(instances
+			(project "arduino_brainmachine"
+				(path "/16427a71-30ca-4ef8-b47f-54137aef95d2"
+					(page "2")
+				)
+			)
+		)
+	)
 	(sheet_instances
 		(path "/"
-			(page "1")
+			(page "2")
 		)
 	)

Commit message: Upgarde
Parts:
- removed C6, C8: 1 mkF, symbol PCM_Elektuur:C
- removed D3: 12 v, symbol Device:D_Zener
- removed Q3: 2N5551, Package_TO_SOT_THT:TO-39-3, symbol Transistor_BJT:2N2219
- added 12V, 5.1V: ${SIM.PARAMS}, symbol PCM_Elektuur:D-Zener
- added C11, C12, C14, C15, C18: 100nF, symbol PCM_Elektuur:C
- added C13, C6: 220mkF, symbol PCM_Elektuur:C-polar
- added C16: 47mkF, symbol PCM_Elektuur:C-polar
- added C17: 220nF, symbol PCM_Elektuur:C
- added C8: 10mkF, symbol PCM_Elektuur:C-polar
- added D3: LED, symbol Device:LED
- added L1: 10mkH, symbol PCM_Elektuur:L
- added R37, R38: 220 Om, symbol PCM_Elektuur:R
- added R39: 1kOm, symbol PCM_Elektuur:R
- added U3: LM358_DFN, Package_DFN_QFN:DFN-8-1EP_2x2mm_P0.5mm_EP1.05x1.75mm, symbol Amplifier_Operational:LM358_DFN
- added U4: LM7805_TO220, Package_TO_SOT_THT:TO-220-3_Vertical, symbol Regulator_Linear:LM7805_TO220
- R24: value 330 Om -> 1 KOm
- R25: value 200 Om -> 10 KOm
- R26: value 2 KOm -> 10 KOm
- R27: value 1.2 KOm -> 10 KOm
- R28: value 30-56 KOm -> 5-10 KOm
- R29: value 4.7 Om -> 10 KOm
Connections:
- net +12V: now also 12V.1 (K-), C17.1 (+), U4.1 (VI); no longer R26.2 (-), R27.1 (+), R28.2 (-)
- net +5V: now also R26.1 (+), R27.1 (+), R28.2 (-), C11.1 (+), C12.1 (+), C15.1 (+), C16.1 (+), L1.1 (+)
- net GND: now also R25.2 (-), R29.2 (-), 12V.2 (A+), 5.1V.2 (A+), C11.2 (-), C13.2 (-), C15.2 (-), C16.2 (-), C17.2 (-), C18.2 (-), R37.2 (-), R38.2 (-), R39.1 (+), U4.2 (GND); no longer R24.1 (+), R25.1 (+)
- net at MK1.2 (+), R28.1 (+): now also C8.1 (+)
- net at R24.2 (-): now also U3.2 (-); no longer R26.1 (+)
- net at RV1.2, RV1.3, RV2.1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: now also A1.A1; no longer A1.A0
- net at RV3.2, RV3.3, RV4.1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: now also A1.A2; no longer A1.A1
- net at R27.2 (-), R29.1 (+): now also U3.5 (+)
- new net: C12.2 (-), R37.1 (+)
- new net: 5.1V.1 (K-), C13.1 (+), C14.1 (+), C18.1 (+), D3.2 (A), L1.2 (-), U4.3 (VO)
- new net: A1.A0, U3.7
- new net: C6.2 (-), U3.6 (-)
- new net: C6.1 (+), U3.1
- new net: D3.1 (K), R39.2 (-)
- new net: C8.2 (-), R24.1 (+)
- new net: R25.1 (+), R26.2 (-), U3.3 (+)
- new net: C14.2 (-), R38.1 (+)
Other:
- note added: "Use ADC Power Connections If possible To AVCC pin on Atmega328"
- moved on the sheet: MK1, R28

Commit message: Upgrade schematics
Parts:
- added D5: LED, symbol Device:LED
- added R40: 10kOm, symbol PCM_Elektuur:R
Connections:
- net +12V: now also D5.2 (A)
- net GND: now also R40.1 (+)
- net at A1.D3 (D3_INT1): now also R30.1 (+)
- new net: D5.1 (K), R40.2 (-)
- new net: A1.D5, R1.2 (-)
- now unconnected: A1.D4, A1.D6, R2.2 (-)
Changed lines of the file:
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@@
 	)
 	(junction
+		(at 179.07 55.88)
+		(diameter 0)
+		(color 0 0 0 0)
+	)
+	(junction
 		(at 21.59 41.91)
 		(diameter 0)
@@
 	)
 	(junction
+		(at 151.13 35.56)
+		(diameter 0)
+		(color 0 0 0 0)
+	)
+	(junction
 		(at 196.85 133.35)
 		(diameter 0)
@@
 	)
 	(junction
+		(at 163.83 92.71)
+		(diameter 0)
+		(color 0 0 0 0)
+	)
+	(junction
 		(at 40.64 76.2)
 		(diameter 0)
@@
 	)
 	(junction
-		(at 149.86 40.64)
-		(diameter 0)
-		(color 0 0 0 0)
-	)
-	(junction
 		(at 241.3 125.73)
 		(diameter 0)
@@
 	)
 	(junction
-		(at 149.86 38.1)
-		(diameter 0)
-		(color 0 0 0 0)
-	)
-	(junction
 		(at 229.87 116.84)
 		(diameter 0)
@@
 	)
 	(junction
-		(at 148.59 38.1)
-		(diameter 0)
-		(color 0 0 0 0)
-	)
-	(junction
 		(at 252.73 125.73)
 		(diameter 0)
@@
 	(wire
 		(pts
-			(xy 148.59 38.1) (xy 144.78 38.1)
+			(xy 163.83 81.28) (xy 163.83 83.82)
 		)
 		(stroke
@@
 	(wire
 		(pts
+			(xy 151.13 35.56) (xy 151.13 38.1)
+		)
+		(stroke
+			(width 0)
+			(type default)
+		)
+	)
+	(wire
+		(pts
 			(xy 19.05 144.78) (xy 19.05 151.13)
 		)
@@
 	(wire
 		(pts
-			(xy 148.59 38.1) (xy 148.59 43.18)
-		)
-		(stroke
-			(width 0)
-			(type default)
-		)
-	)
-	(wire
-		(pts
 			(xy 207.01 107.95) (xy 207.01 115.57)
 		)
@@
 	(wire
 		(pts
-			(xy 149.86 35.56) (xy 152.4 35.56)
-		)
-		(stroke
-			(width 0)
-			(type default)
-		)
-	)
-	(wire
-		(pts
 			(xy 250.19 96.52) (xy 250.19 101.6)
 		)
@@
 	(wire
 		(pts
-			(xy 149.86 35.56) (xy 149.86 38.1)
+			(xy 53.34 41.91) (xy 53.34 40.64)
 		)
 		(stroke
@@
 	(wire
 		(pts
-			(xy 53.34 41.91) (xy 53.34 40.64)
+			(xy 276.86 125.73) (xy 276.86 120.65)
 		)
 		(stroke
@@
 	(wire
 		(pts
-			(xy 276.86 125.73) (xy 276.86 120.65)
+			(xy 16.51 121.92) (xy 16.51 123.19)
 		)
 		(stroke
@@
 	(wire
 		(pts
-			(xy 16.51 121.92) (xy 16.51 123.19)
+			(xy 240.03 125.73) (xy 241.3 125.73)
 		)
 		(stroke
@@
 	(wire
 		(pts
-			(xy 240.03 125.73) (xy 241.3 125.73)
+			(xy 252.73 154.94) (xy 252.73 156.21)
 		)
 		(stroke
@@
 	(wire
 		(pts
-			(xy 252.73 154.94) (xy 252.73 156.21)
+			(xy 179.07 64.77) (xy 179.07 55.88)
 		)
 		(stroke
@@
 	(wire
 		(pts
+			(xy 163.83 91.44) (xy 163.83 92.71)
+		)
+		(stroke
+			(width 0)
+			(type default)
+		)
+	)
+	(wire
+		(pts
 			(xy 30.48 29.21) (xy 38.1 29.21)
 		)
@@
 	(wire
 		(pts
-			(xy 151.13 38.1) (xy 149.86 38.1)
-		)
-		(stroke
-			(width 0)
-			(type default)
-		)
-	)
-	(wire
-		(pts
 			(xy 203.2 140.97) (xy 210.82 140.97)
 		)
@@
 	(wire
 		(pts
-			(xy 149.86 38.1) (xy 148.59 38.1)
-		)
-		(stroke
-			(width 0)
-			(type default)
-		)
-	)
-	(wire
-		(pts
 			(xy 69.85 127) (xy 78.74 127)
 		)
@@
 	(wire
 		(pts
-			(xy 151.13 16.51) (xy 151.13 38.1)
+			(xy 151.13 16.51) (xy 151.13 35.56)
 		)
 		(stroke
@@
 	(wire
 		(pts
+			(xy 163.83 71.12) (xy 163.83 64.77)
+		)
+		(stroke
+			(width 0)
+			(type default)
+		)
+	)
+	(wire
+		(pts
 			(xy 252.73 125.73) (xy 252.73 144.78)
 		)
@@
 	(wire
 		(pts
+			(xy 144.78 35.56) (xy 151.13 35.56)
+		)
+		(stroke
+			(width 0)
+			(type default)
+		)
+	)
+	(wire
+		(pts
 			(xy 163.83 194.31) (xy 163.83 196.85)
 		)
@@
 	(wire
 		(pts
-			(xy 163.83 92.71) (xy 163.83 97.79)
-		)
-		(stroke
-			(width 0)
-			(type default)
-		)
-	)
-	(wire
-		(pts
 			(xy 170.18 46.99) (xy 205.74 46.99)
 		)
@@
 	(wire
 		(pts
+			(xy 163.83 64.77) (xy 179.07 64.77)
+		)
+		(stroke
+			(width 0)
+			(type default)
+		)
+	)
+	(wire
+		(pts
 			(xy 212.09 88.9) (xy 212.09 90.17)
 		)
@@
 	(wire
 		(pts
+			(xy 163.83 92.71) (xy 163.83 97.79)
+		)
+		(stroke
+			(width 0)
+			(type default)
+		)
+	)
+	(wire
+		(pts
 			(xy 241.3 68.58) (xy 224.79 68.58)
 		)
@@
 	(wire
 		(pts
-			(xy 149.86 40.64) (xy 149.86 38.1)
-		)
-		(stroke
-			(width 0)
-			(type default)
-		)
-	)
-	(wire
-		(pts
 			(xy 170.18 59.69) (xy 185.42 59.69)
 		)
@@
 	)
 	(symbol
+		(lib_id "PCM_Elektuur:R")
+		(at 163.83 76.2 0)
+		(unit 1)
+		(exclude_from_sim no)
+		(in_bom yes)
+		(on_board yes)
+		(dnp no)
+		(fields_autoplaced yes)
+		(property "Reference" "R40"
+			(at 166.37 74.9299 0)
+			(effects
+				(font
+					(size 1.27 1.27)
+				)
+				(justify left)
+			)
+		)
+		(property "Value" "10kOm"
+			(at 166.37 77.4699 0)
+			(effects
+				(font
+					(size 1.27 1.27)
+				)
+				(justify left)
+			)
+		)
+		(property "Footprint" ""
+			(at 163.83 76.2 0)
+			(effects
+				(font
+					(size 1.27 1.27)
+				)
+				(hide yes)
+			)
+		)
+		(property "Datasheet" ""
+			(at 163.83 76.2 0)
+			(effects
+				(font
+					(size 1.27 1.27)
+				)
+				(hide yes)
+			)
+		)
+		(property "Description" "resistor"
+			(at 163.83 76.2 0)
+			(effects
+				(font
+					(size 1.27 1.27)
+				)
+				(hide yes)
+			)
+		)
+		(property "Indicator" "+"
+			(at 160.655 73.025 0)
+			(effects
+				(font
+					(size 1.27 1.27)
+				)
+				(hide yes)
+			)
+		)
+		(property "Rating" "W"
+			(at 166.37 79.375 0)
+			(effects
+				(font
+					(size 1.27 1.27)
+				)
+				(justify left)
+				(hide yes)
+			)
+		)
+		(pin "2"
+		)
+		(pin "1"
+		)
+		(instances
+			(project "arduino_brainmachine"
+				(path "/16427a71-30ca-4ef8-b47f-54137aef95d2"
+					(reference "R40")
+					(unit 1)
+				)
+			)
+		)
+	)
+	(symbol
 		(lib_id "PCM_Elektuur:C")
 		(at 252.73 63.5 0)
@@
 					(unit 1)
 				)
+			)
+		)
+	)
+	(symbol
+		(lib_id "Device:LED")
+		(at 163.83 87.63 270)
+		(unit 1)
+		(exclude_from_sim no)
+		(in_bom yes)
+		(on_board yes)
+		(dnp no)
+		(fields_autoplaced yes)
+		(property "Reference" "D5"
+			(at 166.37 84.7724 90)
+			(effects
+				(font
+					(size 1.27 1.27)
+				)
+				(justify left)
+			)
+		)
+		(property "Value" "LED"
+			(at 166.37 87.3124 90)
+			(effects
+				(font
+					(size 1.27 1.27)
+				)
+				(justify left)
+			)
+		)
+		(property "Footprint" ""
+			(at 163.83 87.63 0)
+			(effects
+				(font
+					(size 1.27 1.27)
+				)
+				(hide yes)
+			)
+		)
+		(property "Datasheet" "~"
+			(at 163.83 87.63 0)
+			(effects
+				(font
+					(size 1.27 1.27)
+				)
+				(hide yes)
+			)
+		)
+		(property "Description" "Light emitting diode"
+			(at 163.83 87.63 0)
+			(effects
+				(font
+					(size 1.27 1.27)
+				)
+				(hide yes)
+			)
+		)
+		(pin "2"
+		)
+		(pin "1"
+		)
+		(instances
+			(project ""
+				(path "/16427a71-30ca-4ef8-b47f-54137aef95d2"
+					(reference "D5")
+					(unit 1)
+				)

Commit message: Upgrade schematics | fixed
Parts:
- added R41, R42: 100 KOm, symbol PCM_Elektuur:R
Connections:
- net +5V: now also A1.5V4 (5V), D1.2 (A), D2.2 (A), Q5.3 (E), Q6.3 (E), U1.1, U2.1
- net at A1.A0, U3.7: now also R42.1 (+)
- net at A1.D5: now also R2.2 (-); no longer R1.2 (-)
- net at A1.D6: now also R1.2 (-)
- net at C6.2 (-), U3.6 (-): now also R42.2 (-)
- net at C6.1 (+), U3.1: now also R41.2 (-)
- net at R24.2 (-), U3.2 (-): now also R41.1 (+)

Commit message: Upgrade schematics | fixed
Parts:
- R40: value 10kOm -> 5-10kOm
Connections:
- net +12V: now also R40.2 (-); no longer D5.2 (A)
- net GND: now also D3.1 (K), D5.1 (K); no longer R39.1 (+), R40.1 (+)
- net at 5.1V.1 (K-), C13.1 (+), C14.1 (+)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: now also R39.2 (-); no longer D3.2 (A)
- new net: D5.2 (A), R40.1 (+)
- new net: D3.2 (A), R39.1 (+)
Other:
- moved on the sheet: D5, R39

Commit message: Upgrade schematics | fixed
Parts:
- added R43: 9.8 KOm, symbol PCM_Elektuur:R
Connections:
- net +5V: now also R43.2 (-)
- net at A1.AREF: now also R43.1 (+)
Changed lines of the file:
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@@
 	)
 	(junction
+		(at 53.34 121.92)
+		(diameter 0)
+		(color 0 0 0 0)
+	)
+	(junction
 		(at 29.21 41.91)
 		(diameter 0)
@@
 	(wire
 		(pts
+			(xy 63.5 109.22) (xy 63.5 106.68)
+		)
+		(stroke
+			(width 0)
+			(type default)
+		)
+	)
+	(wire
+		(pts
 			(xy 16.51 121.92) (xy 16.51 123.19)
 		)
@@
 	(wire
 		(pts
+			(xy 63.5 106.68) (xy 78.74 106.68)
+		)
+		(stroke
+			(width 0)
+			(type default)
+		)
+	)
+	(wire
+		(pts
+			(xy 53.34 121.92) (xy 63.5 121.92)
+		)
+		(stroke
+			(width 0)
+			(type default)
+		)
+	)
+	(wire
+		(pts
 			(xy 44.45 148.59) (xy 46.99 148.59)
 		)
@@
 	(wire
 		(pts
+			(xy 52.07 121.92) (xy 53.34 121.92)
+		)
+		(stroke
+			(width 0)
+			(type default)
+		)
+	)
+	(wire
+		(pts
 			(xy 144.78 43.18) (xy 149.86 43.18)
 		)
@@
 	(wire
 		(pts
+			(xy 63.5 119.38) (xy 63.5 121.92)
+		)
+		(stroke
+			(width 0)
+			(type default)
+		)
+	)
+	(wire
+		(pts
 			(xy 210.82 140.97) (xy 226.06 140.97)
 		)
@@
 	(wire
 		(pts
-			(xy 53.34 121.92) (xy 52.07 121.92)
-		)
-		(stroke
-			(width 0)
-			(type default)
-		)
-	)
-	(wire
-		(pts
 			(xy 166.37 196.85) (xy 163.83 196.85)
 		)
@@
 					(unit 1)
 				)
+			)
+		)
+	)
+	(symbol
+		(lib_id "PCM_Elektuur:R")
+		(at 63.5 114.3 0)
+		(unit 1)
+		(exclude_from_sim no)
+		(in_bom yes)
+		(on_board yes)
+		(dnp no)
+		(fields_autoplaced yes)
+		(property "Reference" "R43"
+			(at 66.04 113.0299 0)
+			(effects
+				(font
+					(size 1.27 1.27)
+				)
+				(justify left)
+			)
+		)
+		(property "Value" "9.8 KOm"
+			(at 66.04 115.5699 0)
+			(effects
+				(font
+					(size 1.27 1.27)
+				)
+				(justify left)
+			)
+		)
+		(property "Footprint" ""
+			(at 63.5 114.3 0)
+			(effects
+				(font
+					(size 1.27 1.27)
+				)
+				(hide yes)
+			)
+		)
+		(property "Datasheet" ""
+			(at 63.5 114.3 0)
+			(effects
+				(font
+					(size 1.27 1.27)
+				)
+				(hide yes)
+			)
+		)
+		(property "Description" "resistor"
+			(at 63.5 114.3 0)
+			(effects
+				(font
+					(size 1.27 1.27)
+				)
+				(hide yes)
+			)
+		)
+		(property "Indicator" "+"
+			(at 60.325 111.125 0)
+			(effects
+				(font
+					(size 1.27 1.27)
+				)
+				(hide yes)
+			)
+		)
+		(property "Rating" "W"
+			(at 66.04 117.475 0)
+			(effects
+				(font
+					(size 1.27 1.27)
+				)
+				(justify left)
+				(hide yes)
+			)
+		)
+		(pin "2"
+		)
+		(pin "1"
+		)
+		(instances
+			(project "arduino_brainmachine"
+				(path "/16427a71-30ca-4ef8-b47f-54137aef95d2"
+					(reference "R43")
+					(unit 1)
+				)

Commit message: Upgrade
Parts:
- removed U1, U2: VOS618A, Package_SO:SSOP-4_4.4x2.6mm_P1.27mm, symbol Isolator:VOS618A
- added C19: 1mkF, symbol PCM_Elektuur:C-polar
- added C20: 10nF, symbol PCM_Elektuur:C
- added D6, D7: LED, symbol Device:LED
- added P1, P2, P3, P4: P-trim, symbol PCM_Elektuur:P-trim
- added Q3, Q7, Q8, Q9: PNP, symbol Simulation_SPICE:PNP
- added R44, R45, R46, R47: 220 Om, symbol PCM_Elektuur:R
- added U1: NE555P, Package_DIP:DIP-8_W7.62mm, symbol Timer:NE555P
Connections:
- net +5V: now also P2.3 (c), P3.3 (c), Q3.3 (E), R46.2 (-), U1.4 (R), U1.8 (VCC)
- net GND: now also C19.2 (-), C20.2 (-), D6.1 (K), D7.1 (K), U1.1 (GND)
- net at R36.2 (-): now also Q7.2 (B); no longer Q6.2 (B)
- net at R35.2 (-): now also Q8.2 (B); no longer Q5.2 (B)
- new net: D7.2 (A), R44.1 (+)
- new net: P3.1 (a), P3.2 (b), P4.1 (a), P4.2 (b), Q8.1 (C)
- new net: Q8.3 (E), Q9.2 (B), R47.1 (+)
- new net: Q3.1 (C), R44.2 (-)
- new net: Q9.3 (E), R47.2 (-), U1.7 (DIS)
- new net: P1.1 (a), P1.2 (b), P2.1 (a), P2.2 (b), Q9.1 (C)
- new net: Q3.2 (B), Q7.3 (E), R46.1 (+)
- new net: D6.2 (A), R45.1 (+)
- new net: Q7.1 (C), R45.2 (-)
- new net: C19.1 (+), U1.2 (TR)
- new net: P1.3 (c), P4.3 (c), U1.6 (THR)
- new net: C20.1 (+), U1.5 (CV)
Other:
- moved on the sheet: Q5, Q6

Commit message: Upgrade
Other:
- note added: "TEST"
Changed lines of the file:
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@@
+		)
+	)
+	(text "TEST"
+		(exclude_from_sim no)
+		(at 42.672 213.36 0)
+		(effects
+			(font
+				(size 1.27 1.27)
+			)
 		)
 	)
